Commit message: urdf inertia

File: uniteedog_description/urdf/unitreeDog.urdf (robot description, URDF)
Before this commit: robot UnitreeDog, 15 links, 14 joints
Links:
- link back_calf_left: mass None -> 0.6; geometry collision cylinder length=0.14 radius=0.025; visual mesh filename=package://uniteedog_description/meshes/calf.dae scale=1.0 1.0 1.0
- link back_calf_right: mass None -> 0.6; geometry collision cylinder length=0.14 radius=0.025; visual mesh filename=package://uniteedog_description/meshes/calf.dae scale=1.0 1.0 1.0
- link back_hip_left: mass None -> 0.125; geometry collision box size=0.06 0.04 0.04; visual mesh filename=package://uniteedog_description/meshes/hip.dae scale=1.0 1.0 1.0
- link back_hip_right: mass None -> 0.125; geometry collision box size=0.06 0.04 0.04; visual mesh filename=package://uniteedog_description/meshes/hip.dae scale=1.0 1.0 1.0
- link base_link: mass None -> 5.5; geometry collision box size=0.588 0.22 0.12; visual mesh filename=package://uniteedog_description/meshes/trunk.dae scale=1.0 1.0 1.0
- link camera: mass None -> 0.15; geometry collision box size=0.08 0.03 0.03; visual mesh filename=package://uniteedog_description/meshes/depthCamera.dae scale=1.0 1.0 1.0
- link front_calf_left: mass None -> 0.6; geometry collision cylinder length=0.14 radius=0.025; visual mesh filename=package://uniteedog_description/meshes/calf.dae scale=1.0 1.0 1.0
- link front_calf_right: mass None -> 0.6; geometry collision cylinder length=0.14 radius=0.025; visual mesh filename=package://uniteedog_description/meshes/calf.dae scale=1.0 1.0 1.0
- link front_hip_left: mass None -> 0.125; geometry collision box size=0.06 0.04 0.04; visual mesh filename=package://uniteedog_description/meshes/hip.dae scale=1.0 1.0 1.0
- link front_hip_right: mass None -> 0.125; geometry collision box size=0.06 0.04 0.04; visual mesh filename=package://uniteedog_description/meshes/hip.dae scale=1.0 1.0 1.0
- link left_back_leg: mass None -> 0.9; geometry collision cylinder length=0.12 radius=0.03; visual mesh filename=package://uniteedog_description/meshes/thigh.dae scale=1.0 1.0 1.0
- link left_front_leg: mass None -> 0.9; geometry collision cylinder length=0.12 radius=0.03; visual mesh filename=package://uniteedog_description/meshes/thigh.dae scale=1.0 1.0 1.0
- link right_back_leg: mass None -> 0.9; geometry collision cylinder length=0.12 radius=0.03; visual mesh filename=package://uniteedog_description/meshes/thigh_mirror.dae scale=1.0 1.0 1.0
- link right_front_leg: mass None -> 0.9; geometry collision cylinder length=0.12 radius=0.03; visual mesh filename=package://uniteedog_description/meshes/thigh_mirror.dae scale=1.0 1.0 1.0
- link ultraSound: mass None -> 0.05; geometry collision box size=0.04 0.02 0.02; visual mesh filename=package://uniteedog_description/meshes/ultraSound.dae scale=1.0 1.0 1.0
Joints:
- joint base_to_left_front_leg: origin xyz=0 0.08 0  rpy=0 0 0 -> xyz=0 0.08 0 rpy=0 0 0
- joint hip_to_left_back_leg: origin xyz=0 0.08 0  rpy=0 0 0 -> xyz=0 0.08 0 rpy=0 0 0
- joint hip_to_right_back_leg: origin xyz=0 -0.08 0  rpy=0 0 0 -> xyz=0 -0.08 0 rpy=0 0 0
- joint left_back_leg_to_calf: origin xyz= -0.14 0 -0.15  rpy=0 -0.7854 0 -> xyz=-0.14 0 -0.15 rpy=0 -0.7854 0
- joint left_front_leg_to_calf: origin xyz= -0.14 0 -0.15  rpy=0 -0.7854 0 -> xyz=-0.14 0 -0.15 rpy=0 -0.7854 0
- joint right_back_leg_to_calf: origin xyz= -0.14 0 -0.15  rpy=0 -0.7854 0 -> xyz=-0.14 0 -0.15 rpy=0 -0.7854 0
- joint right_front_leg_to_calf: origin xyz= -0.14 0 -0.15  rpy=0 -0.7854 0 -> xyz=-0.14 0 -0.15 rpy=0 -0.7854 0
