Commit message: fix: resolve missing legs in RViz by adding joint_state_publisher

File: unitreedog_description/urdf/unitreeDog.urdf.xacro (robot description, xacro)
@@ -173,57 +173,6 @@
        CAMERA (small mass)
        =========================== -->
-  <link name="camera">
-    <visual>
-      <origin xyz="0 -0.01 0.01" rpy="0.7854 0 0"/>
-      <geometry>
-        <mesh filename="package://unitreedog_description/meshes/depthCamera.dae" scale="1.0 1.0 1.0"/>
-      </geometry>
-      <material name="base_color">
-        <color rgba="0.9 0.29 0.0 1"/>
-      </material>
-    </visual>
-    <collision>
-      <origin xyz="0 0 0" rpy="0 0 0"/>
-      <geometry>
-        <box size="0.08 0.03 0.03"/>
-      </geometry>
-    </collision>
-    <inertial>
-      <origin xyz="0 0 0" rpy="0 0 0"/>
-      <mass value="0.15"/>
-      <!-- approx sphere inertia (r~0.03) -->
-      <inertia
-        ixx="0.000054" ixy="0.0" ixz="0.0"
-        iyy="0.000054" iyz="0.0"
-        izz="0.000054"/>
-    </inertial>
-    <sensor name="unitree_camera" type="camera">
-    <pose>0 0 0 0 0 0</pose>
-    <visualize>true</visualize>
-    <update_rate>30</update_rate>
-    <camera>
-      <horizontal_fov>1.089</horizontal_fov>
-      <image>
-        <width>640</width>
-        <height>480</height>
-        <format>R8G8B8</format>
-      </image>
-      <clip>
-        <near>0.05</near>
-        <far>8.0</far>
-      </clip>
-    </camera>
-    <topic>camera/image_raw</topic>
-    <plugin
-      filename="ignition-gazebo-camera-plugin"
-      name="ignition::gazebo::systems::Camera">
-    </plugin>
-  </sensor>
-  </link>
-  <joint name="base_to_camera" type="fixed">
-    <parent link="base_link"/>
-    <child link="camera"/>
-    <origin xyz="0.3 0 0" rpy="0 0 0"/>
-  </joint>
+    <xacro:include filename="$(find unitreedog_description)/urdf/camera.urdf.xacro"/>
+    <xacro:camera parent="base_link"/>
   <!-- ===========================
        ULTRASOUND SENSOR
@@ -255,5 +204,5 @@
   </link>
   <joint name="base_to_ultraSound" type="fixed">
-    <parent link="camera"/>
+    <parent link="camera_link"/>
     <child link="ultraSound"/>
     <origin xyz="0 0 0" rpy="0 0 0"/>
@@ -272,11 +221,10 @@
       </material>
     </visual>
-    <collision>
-      <origin xyz="0 0 0" rpy="0 0 0"/>
-      <geometry>
-        <!-- cylinder: length ~0.12 m, radius 0.03 m (aligned along local X) -->
+    <!-- <collision>
+      <origin xyz="0 0 0" rpy="0 0 0"/>
+      <geometry>
         <cylinder length="0.12" radius="0.03"/>
       </geometry>
-    </collision>
+    </collision> -->
     <inertial>
       <origin xyz="0 0 0" rpy="0 0 0"/>
@@ -307,11 +255,10 @@
       </material>
     </visual>
-    <collision>
-      <origin xyz="0 0 0" rpy="0 0 0"/>
-      <geometry>
-        <!-- cylinder: length 0.14 m, radius 0.025 m -->
+    <!-- <collision>
+      <origin xyz="0 0 0" rpy="0 0 0"/>
+      <geometry>
         <cylinder length="0.14" radius="0.025"/>
       </geometry>
-    </collision>
+    </collision> -->
     <inertial>
       <origin xyz="0 0 0" rpy="0 0 0"/>
@@ -345,10 +292,10 @@
       </material>
     </visual>
-    <collision>
+    <!-- <collision>
       <origin xyz="0 0 0" rpy="0 0 0"/>
       <geometry>
         <cylinder length="0.12" radius="0.03"/>
       </geometry>
-    </collision>
+    </collision> -->
     <inertial>
       <origin xyz="0 0 0" rpy="0 0 0"/>
@@ -377,10 +324,10 @@
       </material>
     </visual>
-    <collision>
+    <!-- <collision>
       <origin xyz="0 0 0" rpy="0 0 0"/>
       <geometry>
         <cylinder length="0.14" radius="0.025"/>
       </geometry>
-    </collision>
+    </collision> -->
     <inertial>
       <origin xyz="0 0 0" rpy="0 0 0"/>
@@ -412,10 +359,10 @@
       </material>
     </visual>
-    <collision>
+    <!-- <collision>
       <origin xyz="0 0 0" rpy="0 0 0"/>
       <geometry>
         <cylinder length="0.12" radius="0.03"/>
       </geometry>
-    </collision>
+    </collision> -->
     <inertial>
       <origin xyz="0 0 0" rpy="0 0 0"/>
@@ -444,10 +391,10 @@
       </material>
     </visual>
-    <collision>
+    <!-- <collision>
       <origin xyz="0 0 0" rpy="0 0 0"/>
       <geometry>
         <cylinder length="0.14" radius="0.025"/>
       </geometry>
-    </collision>
+    </collision> -->
     <inertial>
       <origin xyz="0 0 0" rpy="0 0 0"/>
@@ -479,10 +426,10 @@
       </material>
     </visual>
-    <collision>
+    <!-- <collision>
       <origin xyz="0 0 0" rpy="0 0 0"/>
       <geometry>
         <cylinder length="0.12" radius="0.03"/>
       </geometry>
-    </collision>
+    </collision> -->
     <inertial>
       <origin xyz="0 0 0" rpy="0 0 0"/>
@@ -511,10 +458,10 @@
       </material>
     </visual>
-    <collision>
+    <!-- <collision>
       <origin xyz="0 0 0" rpy="0 0 0"/>
       <geometry>
         <cylinder length="0.14" radius="0.025"/>
       </geometry>
-    </collision>
+    </collision> -->
     <inertial>
       <origin xyz="0 0 0" rpy="0 0 0"/>
@@ -533,33 +480,3 @@
     <origin xyz="-0.14 0 -0.15" rpy="0 -0.7854 0"/>
   </joint>
-  <!-- <gazebo>
-  <plugin name="ros2_control" filename="libignition_ros2_control.so">
-    <ros2_control>
-      <robot_namespace>/</robot_namespace>
-      <robot_sim_type>gazebo_ros2_control/DefaultRobotHWSim</robot_sim_type>
-    </ros2_control>
-  </plugin>
-  <plugin name="camera" filename="libignition_ros_camera_sensor.so">
-    <ros>
-      <namespace>/camera</namespace>
-    </ros>
-    <sensorName>unitree_camera</sensorName>
-    <topic>/camera/image_raw</topic>
-    <updateRate>30</updateRate>
-  </plugin>
-</gazebo> -->
-<gazebo>
-  <plugin
-    filename="ign_ros2_control-system"
-    name="ign_ros2_control::IgnitionRos2ControlSystem">
-    <ros>
-      <namespace>/</namespace>
-    </ros>
-    </plugin>
-  <plugin
-    filename="ignition-gazebo-sensors-system"
-    name="ignition::gazebo::systems::Sensors">
-    <render_engine>ogre2</render_engine>
-  </plugin>
-</gazebo>
 </robot>

Commit message: fix: URDF parsing errors

File: unitreedog_description/urdf/unitreeDog.urdf.xacro (robot description, xacro)
@@ -1,482 +1,225 @@
+<?xml version="1.0"?>
 <robot name="UnitreeDog" xmlns:xacro="http://www.ros.org/wiki/xacro">
-  <!-- ===========================
-       BASE / TRUNK (box approx)
-       =========================== -->
+  <!-- BASE LINK -->
   <link name="base_link">
     <visual>
-      <origin xyz="0 0 0" rpy="0 0 0"/>
-      <geometry>
-        <mesh filename="package://unitreedog_description/meshes/trunk.dae" scale="1.0 1.0 1.0"/>
-      </geometry>
-      <material name="base_color">
-        <color rgba="0.59 0.29 0.0 1.0"/>
-      </material>
-    </visual>
-    <!-- Collision: simplified box for performance -->
-    <collision>
-      <origin xyz="0 0 0" rpy="0 0 0"/>
-      <geometry>
-        <box size="0.588 0.22 0.12"/> <!-- length x width x height (m) -->
-      </geometry>
-    </collision>
-    <!-- Inertial: computed for the box geometry -->
-    <!-- <inertial>
-      <origin xyz="0 0 0" rpy="0 0 0"/>
+      <origin xyz="0 0 0.06"/>
+      <geometry>
+        <mesh filename="package://unitreedog_description/meshes/trunk.dae"/>
+      </geometry>
+      <material name="brown">
+        <color rgba="0.6 0.3 0.1 1.0"/>
+      </material>
+    </visual>
+    <collision>
+      <origin xyz="0 0 0.06"/>
+      <geometry>
+        <box size="0.588 0.22 0.12"/>
+      </geometry>
+    </collision>
+    <inertial>
+      <origin xyz="0 0 0.06"/>
       <mass value="5.5"/>
-      <inertia
-        ixx="0.02878333" ixy="0.0" ixz="0.0"
-        iyy="0.16506600" iyz="0.0"
-        izz="0.18064933"/>
-    </inertial> -->
-  </link>
-  <!-- ===========================
-       BACK HIP RIGHT (small block)
-       =========================== -->
+      <inertia ixx="0.02878" iyy="0.16506" izz="0.18064"
+               ixy="0" ixz="0" iyz="0"/>
+    </inertial>
+  </link>
+  <!-- BACK RIGHT HIP -->
   <link name="back_hip_right">
     <visual>
-      <origin xyz="0 0 0" rpy="0 3.1416 0"/>
-      <geometry>
-        <mesh filename="package://unitreedog_description/meshes/hip.dae" scale="1.0 1.0 1.0"/>
-      </geometry>
-      <material name="base_color">
-        <color rgba="0.59 0.29 0.0 1.0"/>
-      </material>
-    </visual>
-    <collision>
-      <origin xyz="0 0 0" rpy="0 0 0"/>
-      <geometry>
-        <box size="0.06 0.04 0.04"/>
-      </geometry>
-    </collision>
-    <inertial>
-      <origin xyz="0 0 0" rpy="0 0 0"/>
-      <mass value="0.125"/>
-      <inertia
-        ixx="0.00003333" ixy="0.0" ixz="0.0"
-        iyy="0.00005417" iyz="0.0"
-        izz="0.00005417"/>
+      <origin rpy="0 3.1416 0"/>
+      <geometry>
+        <mesh filename="package://unitreedog_description/meshes/hip.dae"/>
+      </geometry>
+      <material name="black">
+        <color rgba="0.1 0.1 0.1 1"/>
+      </material>
+    </visual>
+    <collision>
+      <geometry><box size="0.06 0.04 0.04"/></geometry>
+    </collision>
+    <inertial>
+      <mass value="0.125"/>
+      <inertia ixx="0.00003" iyy="0.00005" izz="0.00005"
+               ixy="0" ixz="0" iyz="0"/>
     </inertial>
   </link>
   <joint name="base_to_back_hip_right" type="revolute">
-    <axis xyz="1 0 0"/>
     <parent link="base_link"/>
     <child link="back_hip_right"/>
-    <origin xyz="-0.19 -0.05 0" rpy="0 0 0"/>
-    <limit lower="-0.6" upper="0.6" effort="10" velocity="0.5"/>
-  </joint>
-  <!-- ===========================
-       BACK HIP LEFT
-       =========================== -->
+    <axis xyz="1 0 0"/>
+    <origin xyz="-0.19 -0.05 0.05"/>
+    <limit lower="-0.6" upper="0.6" effort="10" velocity="1.0"/>
+    <dynamics damping="0.5" friction="0.1"/>
+  </joint>
+  <!-- BACK LEFT HIP -->
   <link name="back_hip_left">
     <visual>
-      <origin xyz="0 0 0" rpy="0 3.1416 0"/>
-      <geometry>
-        <mesh filename="package://unitreedog_description/meshes/hip.dae" scale="1.0 1.0 1.0"/>
-      </geometry>
-      <material name="base_color">
-        <color rgba="0.59 0.29 0.0 1.0"/>
-      </material>
-    </visual>
-    <collision>
-      <origin xyz="0 0 0" rpy="0 0 0"/>
-      <geometry>
-        <box size="0.06 0.04 0.04"/>
-      </geometry>
-    </collision>
-    <inertial>
-      <origin xyz="0 0 0" rpy="0 0 0"/>
-      <mass value="0.125"/>
-      <inertia
-        ixx="0.00003333" ixy="0.0" ixz="0.0"
-        iyy="0.00005417" iyz="0.0"
-        izz="0.00005417"/>
+      <origin rpy="0 3.1416 0"/>
+      <geometry>
+        <mesh filename="package://unitreedog_description/meshes/hip.dae"/>
+      </geometry>
+      <material name="black">
+        <color rgba="0.1 0.1 0.1 1"/>
+      </material>
+    </visual>
+    <collision>
+      <geometry><box size="0.06 0.04 0.04"/></geometry>
+    </collision>
+    <inertial>
+      <mass value="0.125"/>
+      <inertia ixx="0.00003" iyy="0.00005" izz="0.00005"
+               ixy="0" ixz="0" iyz="0"/>
     </inertial>
   </link>
   <joint name="base_to_back_hip_left" type="revolute">
-    <axis xyz="1 0 0"/>
     <parent link="base_link"/>
     <child link="back_hip_left"/>
-    <origin xyz="-0.19 0.05 0" rpy="0 0 0"/>
-    <limit lower="-0.6" upper="0.6" effort="10" velocity="0.5"/>
-  </joint>
-  <!-- ===========================
-       FRONT HIP RIGHT
-       =========================== -->
+    <axis xyz="1 0 0"/>
+    <origin xyz="-0.19 0.05 0.05"/>
+    <limit lower="-0.6" upper="0.6" effort="10" velocity="1.0"/>
+    <dynamics damping="0.5" friction="0.1"/>
+  </joint>
+  <!-- FRONT RIGHT HIP -->
   <link name="front_hip_right">
     <visual>
-      <origin xyz="0 0 0" rpy="0 0 0"/>
-      <geometry>
-        <mesh filename="package://unitreedog_description/meshes/hip.dae" scale="1.0 1.0 1.0"/>
-      </geometry>
-      <material name="base_color">
-        <color rgba="0.59 0.29 0.0 1.0"/>
-      </material>
-    </visual>
-    <collision>
-      <origin xyz="0 0 0" rpy="0 0 0"/>
-      <geometry>
-        <box size="0.06 0.04 0.04"/>
-      </geometry>
-    </collision>
-    <inertial>
-      <origin xyz="0 0 0" rpy="0 0 0"/>
-      <mass value="0.125"/>
-      <inertia
-        ixx="0.00003333" ixy="0.0" ixz="0.0"
-        iyy="0.00005417" iyz="0.0"
-        izz="0.00005417"/>
+      <geometry>
+        <mesh filename="package://unitreedog_description/meshes/hip.dae"/>
+      </geometry>
+      <material name="black">
+        <color rgba="0.1 0.1 0.1 1"/>
+      </material>
+    </visual>
+    <collision>
+      <geometry><box size="0.06 0.04 0.04"/></geometry>
+    </collision>
+    <inertial>
+      <mass value="0.125"/>
+      <inertia ixx="0.00003" iyy="0.00005" izz="0.00005"
+               ixy="0" ixz="0" iyz="0"/>
     </inertial>
   </link>
   <joint name="base_to_front_hip_right" type="revolute">
-    <axis xyz="1 0 0"/>
     <parent link="base_link"/>
     <child link="front_hip_right"/>
-    <origin xyz="0.19 -0.05 0" rpy="0 0 0"/>
-    <limit lower="-0.6" upper="0.6" effort="10" velocity="0.5"/>
-  </joint>
-  <!-- ===========================
-       FRONT HIP LEFT
-       =========================== -->
+    <axis xyz="1 0 0"/>
+    <origin xyz="0.19 -0.05 0.05"/>
+    <limit lower="-0.6" upper="0.6" effort="10" velocity="1.0"/>
+    <dynamics damping="0.5" friction="0.1"/>
+  </joint>
+  <!-- FRONT LEFT HIP -->
   <link name="front_hip_left">
     <visual>
-      <origin xyz="0 0 0" rpy="0 0 0"/>
-      <geometry>
-        <mesh filename="package://unitreedog_description/meshes/hip.dae" scale="1.0 1.0 1.0"/>
-      </geometry>
-      <material name="base_color">
-        <color rgba="0.59 0.29 0.0 1.0"/>
-      </material>
-    </visual>
-    <collision>
-      <origin xyz="0 0 0" rpy="0 0 0"/>
-      <geometry>
-        <box size="0.06 0.04 0.04"/>
-      </geometry>
-    </collision>
-    <inertial>
-      <origin xyz="0 0 0" rpy="0 0 0"/>
-      <mass value="0.125"/>
-      <inertia
-        ixx="0.00003333" ixy="0.0" ixz="0.0"
-        iyy="0.00005417" iyz="0.0"
-        izz="0.00005417"/>
+      <geometry>
+        <mesh filename="package://unitreedog_description/meshes/hip.dae"/>
+      </geometry>
+      <material name="black">
+        <color rgba="0.1 0.1 0.1 1"/>
+      </material>
+    </visual>
+    <collision>
+      <geometry><box size="0.06 0.04 0.04"/></geometry>
+    </collision>
+    <inertial>
+      <mass value="0.125"/>
+      <inertia ixx="0.00003" iyy="0.00005" izz="0.00005"
+               ixy="0" ixz="0" iyz="0"/>
     </inertial>
   </link>
   <joint name="base_to_front_hip_left" type="revolute">
-    <axis xyz="1 0 0"/>
     <parent link="base_link"/>
     <child link="front_hip_left"/>
-    <origin xyz="0.19 0.05 0" rpy="0 0 0"/>
-    <limit lower="-0.6" upper="0.6" effort="10" velocity="0.5"/>
-  </joint>
-  <!-- ===========================
-       CAMERA (small mass)
-       =========================== -->
-    <xacro:include filename="$(find unitreedog_description)/urdf/camera.urdf.xacro"/>
-    <xacro:camera parent="base_link"/>
-  <!-- ===========================
-       ULTRASOUND SENSOR
-       =========================== -->
-  <link name="ultraSound">
-    <visual>
-      <origin xyz="0 0 0.02" rpy="-0.7854 0 0"/>
-      <geometry>
-        <mesh filename="package://unitreedog_description/meshes/ultraSound.dae" scale="1.0 1.0 1.0"/>
-      </geometry>
-      <material name="base_color">
-        <color rgba="0.9 0.29 0.0 1"/>
-      </material>
-    </visual>
-    <collision>
-      <origin xyz="0 0 0" rpy="0 0 0"/>
-      <geometry>
-        <box size="0.04 0.02 0.02"/>
-      </geometry>
-    </collision>
-    <inertial>
-      <origin xyz="0 0 0" rpy="0 0 0"/>
-      <mass value="0.05"/>
-      <inertia
-        ixx="0.00001" ixy="0.0" ixz="0.0"
-        iyy="0.00001" iyz="0.0"
-        izz="0.00001"/>
-    </inertial>
-  </link>
-  <joint name="base_to_ultraSound" type="fixed">
-    <parent link="camera_link"/>
-    <child link="ultraSound"/>
-    <origin xyz="0 0 0" rpy="0 0 0"/>
-  </joint>
-  <!-- ===========================
-       RIGHT FRONT THIGH (cylinder)
-       =========================== -->
-  <link name="right_front_leg">
-    <visual>
-      <origin xyz="0 0 0" rpy="0 0.7854 0"/>
-      <geometry>
-        <mesh filename="package://unitreedog_description/meshes/thigh_mirror.dae" scale="1.0 1.0 1.0"/>
-      </geometry>
-      <material name="base_color">
-        <color rgba="0.59 0.29 0.0 1.0"/>
-      </material>
-    </visual>
-    <!-- <collision>
-      <origin xyz="0 0 0" rpy="0 0 0"/>
-      <geometry>
-        <cylinder length="0.12" radius="0.03"/>
-      </geometry>
-    </collision> -->
-    <inertial>
-      <origin xyz="0 0 0" rpy="0 0 0"/>
-      <mass value="0.9"/>
-      <!-- cylinder inertia: I_perp ~0.0012825, I_long ~0.000405 -->
-      <inertia
-        ixx="0.0012825" ixy="0.0" ixz="0.0"
-        iyy="0.0012825" iyz="0.0"
-        izz="0.000405"/>
-    </inertial>
-  </link>
-  <joint name="base_to_right_front_leg" type="revolute">
-    <axis xyz="0 1 0"/>
-    <limit lower="-0.52" upper="1.57" effort="10" velocity="0.5"/>
-    <parent link="front_hip_right"/>
-    <child link="right_front_leg"/>
-    <origin xyz="0 -0.08 0 " rpy="0 0 0"/>
-  </joint>
-  <!-- FRONT CALF RIGHT -->
-  <link name="front_calf_right">
-    <visual>
-      <origin xyz="0 0 0" rpy="0 0 0"/>
-      <geometry>
-        <mesh filename="package://unitreedog_description/meshes/calf.dae" scale="1.0 1.0 1.0"/>
-      </geometry>
-      <material name="base_color">
-        <color rgba="0.59 0.29 0.0 1.0"/>
-      </material>
-    </visual>
-    <!-- <collision>
-      <origin xyz="0 0 0" rpy="0 0 0"/>
-      <geometry>
-        <cylinder length="0.14" radius="0.025"/>
-      </geometry>
-    </collision> -->
-    <inertial>
-      <origin xyz="0 0 0" rpy="0 0 0"/>
-      <mass value="0.6"/>
-      <!-- cylinder inertia: I_perp ~0.00107375, I_long ~0.0001875 -->
-      <inertia
-        ixx="0.00107375" ixy="0.0" ixz="0.0"
-        iyy="0.00107375" iyz="0.0"
-        izz="0.0001875"/>
-    </inertial>
-  </link>
-  <joint name="right_front_leg_to_calf" type="revolute">
-    <axis xyz="0 1 0"/>
-    <limit lower="-1.2" upper="0" effort="10" velocity="0.5"/>
-    <parent link="right_front_leg"/>
-    <child link="front_calf_right"/>
-    <origin xyz="-0.14 0 -0.15" rpy="0 -0.7854 0"/>
-  </joint>
-  <!-- ===========================
-       LEFT FRONT THIGH + CALF
-       (same masses/inertias as right)
-       =========================== -->
-  <link name="left_front_leg">
-    <visual>
-      <origin xyz="0 0 0" rpy="0 0.7854 0"/>
-      <geometry>
-        <mesh filename="package://unitreedog_description/meshes/thigh.dae" scale="1.0 1.0 1.0"/>
-      </geometry>
-      <material name="base_color">
-        <color rgba="0.59 0.29 0.0 1.0"/>
-      </material>
-    </visual>
-    <!-- <collision>
-      <origin xyz="0 0 0" rpy="0 0 0"/>
-      <geometry>
-        <cylinder length="0.12" radius="0.03"/>
-      </geometry>
-    </collision> -->
-    <inertial>
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