Commit message: add PID gains for joint stabilization

File: unitreedog_description/urdf/camera.urdf.xacro (robot description, xacro)
@@ -28,5 +28,32 @@
       <parent link="${parent}"/>
       <child link="camera_link"/>
-      <origin xyz="0.3 0 0" rpy="0 0 0"/>
+      <origin xyz="0.288 0 0.047" rpy="0 0 0"/>
+      <!-- <origin xyz="0.3 0 0" rpy="0 0 0"/> -->
+    </joint>
+    <link name="ultraSound">
+      <visual>
+        <origin xyz="0 0 0.02" rpy="-0.7854 0 0"/>
+        <geometry>
+          <mesh filename="package://unitreedog_description/meshes/ultraSound.dae" scale="1.0 1.0 1.0"/>
+        </geometry>
+        <material name="base_color">
+          <color rgba="0.9 0.29 0.0 1"/>
+        </material>
+      </visual>
+      <inertial>
+        <origin xyz="0 0 0" rpy="0 0 0"/>
+        <mass value="0.15"/>
+        <!-- approx sphere inertia (r~0.03) -->
+        <inertia
+          ixx="0.000054" ixy="0.0" ixz="0.0"
+          iyy="0.000054" iyz="0.0"
+          izz="0.000054"/>
+      </inertial>
+    </link>
+    <joint name="base_to_ultraSound" type="fixed">
+      <parent link="camera_link"/>
+      <child link="ultraSound"/>
+      <origin xyz="0 0 0" rpy="0 0 0"/>
+      <!-- <limit lower="0.0" upper="0.3" effort="10" velocity="0.5"/> -->
     </joint>
     <gazebo reference="camera_link">
@@ -45,5 +72,5 @@
           </clip>
         </camera>
-        <plugin name="camera_controller" filename="libgazebo_ros_camera.so">
+        <plugin name="camera" filename="libgz-sim-camera-system.so">
           <ros>
             <namespace>/camera</namespace>

File: unitreedog_description/urdf/unitreeDog.urdf.xacro (robot description, xacro)
@@ -25,4 +25,7 @@
     </inertial>
   </link>
+   <!-- Camera -->
+  <xacro:include filename="$(find unitreedog_description)/urdf/camera.urdf.xacro"/>
+  <xacro:camera parent="base_link"/>
   <!-- BACK RIGHT HIP -->
   <link name="back_hip_right">
@@ -49,5 +52,5 @@
     <child link="back_hip_right"/>
     <axis xyz="1 0 0"/>
-    <origin xyz="-0.19 -0.05 0.05"/>
+    <origin xyz="-0.19 -0.05 0.06"/>
     <limit lower="-0.6" upper="0.6" effort="10" velocity="1.0"/>
     <dynamics damping="0.5" friction="0.1"/>
@@ -77,5 +80,5 @@
     <child link="back_hip_left"/>
     <axis xyz="1 0 0"/>
-    <origin xyz="-0.19 0.05 0.05"/>
+    <origin xyz="-0.19 0.05 0.06"/>
     <limit lower="-0.6" upper="0.6" effort="10" velocity="1.0"/>
     <dynamics damping="0.5" friction="0.1"/>
@@ -104,5 +107,5 @@
     <child link="front_hip_right"/>
     <axis xyz="1 0 0"/>
-    <origin xyz="0.19 -0.05 0.05"/>
+    <origin xyz="0.19 -0.05 0.06"/>
     <limit lower="-0.6" upper="0.6" effort="10" velocity="1.0"/>
     <dynamics damping="0.5" friction="0.1"/>
@@ -131,5 +134,5 @@
     <child link="front_hip_left"/>
     <axis xyz="1 0 0"/>
-    <origin xyz="0.19 0.05 0.05"/>
+    <origin xyz="0.19 0.05 0.06"/>
     <limit lower="-0.6" upper="0.6" effort="10" velocity="1.0"/>
     <dynamics damping="0.5" friction="0.1"/>
@@ -156,60 +159,60 @@
     </hardware>
     <joint name="base_to_back_hip_right">
-      <command_interface name="effort"/>
+      <command_interface name="position"/>
       <state_interface name="position"/>
       <state_interface name="velocity"/>
     </joint>
     <joint name="base_to_back_hip_left">
-      <command_interface name="effort"/>
+      <command_interface name="position"/>
       <state_interface name="position"/>
       <state_interface name="velocity"/>
     </joint>
     <joint name="base_to_front_hip_right">
-      <command_interface name="effort"/>
+      <command_interface name="position"/>
       <state_interface name="position"/>
       <state_interface name="velocity"/>
     </joint>
     <joint name="base_to_front_hip_left">
-      <command_interface name="effort"/>
+      <command_interface name="position"/>
       <state_interface name="position"/>
       <state_interface name="velocity"/>
     </joint>
     <joint name="base_to_right_front_leg">
-      <command_interface name="effort"/>
+      <command_interface name="position"/>
       <state_interface name="position"/>
       <state_interface name="velocity"/>
     </joint>
     <joint name="right_front_leg_to_calf">
-      <command_interface name="effort"/>
+      <command_interface name="position"/>
       <state_interface name="position"/>
       <state_interface name="velocity"/>
     </joint>
     <joint name="base_to_left_front_leg">
-      <command_interface name="effort"/>
+      <command_interface name="position"/>
       <state_interface name="position"/>
       <state_interface name="velocity"/>
     </joint>
     <joint name="left_front_leg_to_calf">
-      <command_interface name="effort"/>
+      <command_interface name="position"/>
       <state_interface name="position"/>
       <state_interface name="velocity"/>
     </joint>
     <joint name="hip_to_right_back_leg">
-      <command_interface name="effort"/>
+      <command_interface name="position"/>
       <state_interface name="position"/>
       <state_interface name="velocity"/>
     </joint>
     <joint name="right_back_leg_to_calf">
-      <command_interface name="effort"/>
+      <command_interface name="position"/>
       <state_interface name="position"/>
       <state_interface name="velocity"/>
     </joint>
     <joint name="hip_to_left_back_leg">
-      <command_interface name="effort"/>
+      <command_interface name="position"/>
       <state_interface name="position"/>
       <state_interface name="velocity"/>
     </joint>
     <joint name="left_back_leg_to_calf">
-      <command_interface name="effort"/>
+      <command_interface name="position"/>
       <state_interface name="position"/>
       <state_interface name="velocity"/>
